File: Core4GPZ/Core4GPZ.kicad_sch (KiCad schematic)
At the start: 3 parts, among them U1 core4, U2 MPX4250

Commit message: Tiny modification
???
Connections:
- net INJ3_TRIG: no longer names the net of U1.5 (INJ3)
- net INJ4_TRIG: no longer names the net of U1.7 (INJ4)
- no-connect marks 40 -> 42
Changed lines of the file:
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@@
+	)
+	(no_connect
+		(at 50.8 96.52)
 	)
 	(no_connect
@@
 	(no_connect
 		(at 53.34 109.22)
+	)
+	(no_connect
+		(at 50.8 101.6)
 	)
 	(no_connect
@@
 		)
 	)
-	(hierarchical_label "INJ3_TRIG"
-		(shape input)
-		(at 50.8 96.52 180)
-		(fields_autoplaced yes)
-		(effects
-			(font
-				(size 1.27 1.27)
-			)
-			(justify right)
-		)
-	)
 	(hierarchical_label "TACHO"
 		(shape input)
@@
 		)
 	)
-	(hierarchical_label "INJ4_TRIG"
-		(shape input)
-		(at 50.8 101.6 180)
-		(fields_autoplaced yes)
-		(effects
-			(font
-				(size 1.27 1.27)
-			)
-			(justify right)
-		)
-	)
