File: Core4GPZ_rev0-1/inputs.kicad_sch (KiCad schematic)
At the start: 4 parts

Commit message: Reorganised Schematic
Parts:
- added C1: 100uF, Capacitor_SMD:CP_Elec_6.3x7.7, symbol Device:C_Polarized
- added C2: 100nF, Capacitor_SMD:C_0805_2012Metric_Pad1.18x1.45mm_HandSolder, symbol Device:C
- added C3: 1uF, Capacitor_SMD:C_0805_2012Metric_Pad1.18x1.45mm_HandSolder, symbol Device:C
- added JP5: SolderJumper_3_Open, Jumper:SolderJumper-3_P1.3mm_Open_RoundedPad1.0x1.5mm, symbol Jumper:SolderJumper_3_Open
- added JP6: SolderJumper_2_Open, Jumper:SolderJumper-2_P1.3mm_Open_RoundedPad1.0x1.5mm, symbol Jumper:SolderJumper_2_Open
- added R11: 660k, Resistor_SMD:R_0805_2012Metric_Pad1.20x1.40mm_HandSolder, symbol Device:R
- added R12: 300K, Resistor_SMD:R_0805_2012Metric_Pad1.20x1.40mm_HandSolder, symbol Device:R
- added R_CLT1: Thermistor, symbol Device:R
- added U4: LMV321, Package_TO_SOT_SMD:SOT-23-5_HandSoldering, symbol Amplifier_Operational:LMV321
Connections:
- net +5V: now also C2.1, C3.1, U4.5 (V+)
- new net: JP6.2 (B), U4.3 (-), U4.4
- new net: JP5.3 (B), R11.1
- new net: R11.2, R12.1, U4.1 (+)
- new net +12V: C1.1, R_CLT1.1
- new net CLT_5V: JP5.1 (A), JP6.1 (A)
- new net CLT_SNSR: JP5.2 (C), R_CLT1.2
- new net GND: C1.2, C2.2, C3.2, R12.2, U4.2 (V-)
Other:
- note added: "H C"
- note added: "Just a basic filter, for stabilizing the +12v from the bike before feeding it into the CORE4 board. I don't know if it's usefull. *Shrug*"
- note added: "Power Supply"
- note added: "Reference tension for sensors"
- note added: "Temp Gauge (Badly drawn)"
- note added: "Test circuit for decoupling 12V CLT Probe. Convert 12V to 5V, to keep the original instrument working. (Typicaly, the original temperature gauge.)"

Commit message: Updated CAD Enclosure STL and STEP export
Parts:
- D1, D2, D3: footprint Diode_SMD:D_0603_1608Metric -> Diode_SMD:D_0603_1608Metric_Pad1.05x0.95mm_HandSolder
- R1: footprint Resistor_SMD:R_0603_1608Metric -> Resistor_SMD:R_0603_1608Metric_Pad0.98x0.95mm_HandSolder
Changed lines of the file:
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@@
 			)
 		)
-		(property "Footprint" "Resistor_SMD:R_0603_1608Metric"
+		(property "Footprint" "Resistor_SMD:R_0603_1608Metric_Pad0.98x0.95mm_HandSolder"
 			(at 54.102 38.1 90)
 			(effects
@@
 			)
 		)
-		(property "Footprint" "Diode_SMD:D_0603_1608Metric"
+		(property "Footprint" "Diode_SMD:D_0603_1608Metric_Pad1.05x0.95mm_HandSolder"
 			(at 48.26 44.45 0)
 			(effects
@@
 			)
 		)
-		(property "Footprint" "Diode_SMD:D_0603_1608Metric"
+		(property "Footprint" "Diode_SMD:D_0603_1608Metric_Pad1.05x0.95mm_HandSolder"
 			(at 48.26 64.77 0)
 			(effects
@@
 			)
 		)
-		(property "Footprint" "Diode_SMD:D_0603_1608Metric"
+		(property "Footprint" "Diode_SMD:D_0603_1608Metric_Pad1.05x0.95mm_HandSolder"
 			(at 48.26 54.61 0)
 			(effects
