File: Core4GPZ_rev0-1/inputs.kicad_sch (KiCad schematic)
At the start: 13 parts, among them U4 LMV321

Commit message: Updated project library, BOM and documentation
Parts:
- D1, D2, D3: value D -> 1N4448WX-TP; footprint Diode_SMD:D_0603_1608Metric_Pad1.05x0.95mm_HandSolder -> Diode_SMD:D_SOD-323_HandSoldering; Manufacturer (none) -> Micro Commercial Components (MCC); Manufacturer_part (none) -> 1N4448WX-TP; Mouser (none) -> https://www.mouser.fr/ProductDetail/Micro-Commercial-Compon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
- R2: renamed from R1; footprint Resistor_SMD:R_0603_1608Metric_Pad0.98x0.95mm_HandSolder -> Resistor_SMD:R_0805_2012Metric_Pad1.20x1.40mm_HandSolder; Manufacturer (none) -> Yageo; Manufacturer_part (none) -> AC0603FR-7W100KL; Mouser (none) -> https://www.mouser.fr/ProductDetail/YAGEO/AC0603FR-7W100KL
- R3: renamed from R11; Manufacturer (none) -> Yageo; Manufacturer_part (none) -> AC0805FR-07300KL; Mouser (none) -> https://www.mouser.fr/ProductDetail/603-AC0805FR-07300KL
- R4: renamed from R12; Manufacturer (none) -> Yageo; Manufacturer_part (none) -> AC0805FR-07665KL; Mouser (none) -> https://www.mouser.fr/ProductDetail/YAGEO/AC0805FR-07665KL
- renumbered JP5 to JP1, JP6 to JP2
